File: MirageR1.kicad_sch (KiCad schematic)
At the start: 35 parts

Commit message: designed the pcb board w/ a 50x50 mm constrain
Other:
- note added: "TODO: Add switch to prompt connection via BLE. Add 2 LEDs for the eyes. Add LEDs for the top of the board."
Changed lines of the file:
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@@
+    (effects (font (size 1.27 1.27)) (justify left bottom))
+  )
+  (text "TODO:\nAdd switch to prompt connection via BLE.\nAdd 2 LEDs for the eyes.\nAdd LEDs for the top of the board."
+    (at 120.65 154.94 0)
     (effects (font (size 1.27 1.27)) (justify left bottom))
   )

Commit message: finished routing, added gerber files, added footprint positioning file, modified the PCB soldermask, did some bad decisions with my life
Parts:
- removed H? (x4): MountingHole_Pad, symbol Mechanical:MountingHole_Pad
- removed J?: USB_B_Micro, symbol Connector:USB_B_Micro
- removed SW? (x2): SW_Push, Button_Switch_SMD:SW_Push_1P1T_NO_CK_KSC6xxJ, symbol Switch:SW_Push
- added C12, C14, C17, C7: 100n, Capacitor_SMD:C_0402_1005Metric, symbol Device:C_Small
- added D2, D3: Blue, LED_SMD:LED_0805_2012Metric_Pad1.15x1.40mm_HandSolder, symbol Device:LED_Small
- added D4, D5: Emerald, LED_SMD:LED_0805_2012Metric_Pad1.15x1.40mm_HandSolder, symbol Device:LED_Small
- added D6: Red, LED_SMD:LED_0805_2012Metric_Pad1.15x1.40mm_HandSolder, symbol Device:LED_Small
- added D7, D8: White, LED_SMD:LED_0805_2012Metric_Pad1.15x1.40mm_HandSolder, symbol Device:LED_Small
- added J1: USB_B_Mini, Connector_USB:USB_Mini-B_Wuerth_65100516121_Horizontal, symbol Connector:USB_B_Mini
- added R1, R12, R13, R2, R4, R5, R8: 1k, Resistor_SMD:R_0402_1005Metric, symbol Device:R_Small
- added R11: 10k, Resistor_SMD:R_0402_1005Metric, symbol Device:R_Small
- added SW2: SW_Push, Button_Switch_SMD:SW_Push_1P1T_NO_CK_KSC6xxJ, symbol Switch:SW_Push
- C1, C10, C11, C13, C15, C16, C18, C3, C4, C5, C6, C8, C9: renamed from C?; footprint (none) -> Capacitor_SMD:C_0402_1005Metric
- C2: renamed from C?; footprint (none) -> Capacitor_SMD:C_0603_1608Metric
- R10, R14, R3, R6, R7, R9: renamed from R?; footprint (none) -> Resistor_SMD:R_0402_1005Metric
- gave numbers to parts that had none: 8
Connections:
- net PCB_ANT is gone; now on net GND: R14.2
- net +3V3: now also C12.1, C14.1, C17.1, C7.1, SW2.2
- net GND: now also C12.2, C14.2, C7.2, J1.5 (GND), R1.2, R11.2, R12.2, R13.2, R2.2, R4.2, R5.2, R8.2
- net USB_CONN_D+: now also J1.3 (D+)
- net USB_CONN_D-: now also J1.2 (D-)
- net VBUS: now also J1.1 (VBUS)
- net IO25: now reaches U4.14 (IO25)
- net IO25: now also D8.2 (A)
- net IO26: now reaches U4.15 (IO26)
- net IO26: now also C17.2, R11.1, SW2.1
- net IO27: now reaches U4.16 (IO27)
- net IO27: now also D2.2 (A)
- net IO14: now reaches U4.17 (IO14)
- net IO14: now also D4.2 (A)
- net IO12: now reaches U4.18 (IO12)
- net IO12: now also D6.2 (A)
- net IO13: now reaches U4.20 (IO13)
- net IO13: now also D5.2 (A)
- net IO15: now reaches U4.21 (IO15)
- net IO15: now also D3.2 (A)
- net IO4: now reaches U4.24 (IO4)
- net IO4: now also D7.2 (A)
- new net: D4.1 (K), R4.1
- new net: D3.1 (K), R2.1
- new net: D2.1 (K), R1.1
- new net: D5.1 (K), R5.1
- new net: D6.1 (K), R8.1
- new net: D8.1 (K), R13.1
- new net: D7.1 (K), R12.1
- no-connect marks 27 -> 41
Other:
- note added: "BLE Prompt Input"
- note added: "Board LEDs"
- note added: "Eyes LEDs"
- note added: "MCU"
- note added: "There was originally a switch here. The capacitor is used to debounce the switch. I opted to remove them and instead use a pad to connect to an external switch."
- note added: "Used the following datasheets (included the one in the footprint): CP2102-GMR -> https://www.silabs.com/documents/public/data-sheets/CP2102-9.pdf ESP32-DevKitC Schematic -> https://www.espressif.com/en/products/devkits/esp32-devkitc/resources"
- note removed: "Mounting Holes"
- note removed: "TODO: Add switch to prompt connection via BLE. Add 2 LEDs for the eyes. Add LEDs for the top of the board."
- note removed: "Used the following datasheets (included the one in the footprint): CP2102-GMR -> https://www.silabs.com/documents/public/data-sheets/CP2102-9.pdf ESP23-DevKitC Schematic -> https://www.espressif.com/en/products/devkits/esp32-devkitc/resources"
- company: Carlos Vásquez (pions.xyz) -> gluons (pions.xyz)
- moved on the sheet: C10, C11, C13, C15, C16, C18, C3, C4, C5, C6, C8, C9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
